Commit message: moveit config loads, but controllers don't work

File: ur_moveit_config/srdf/ur_macro.srdf.xacro (robot description, xacro)
@@ -13,4 +13,21 @@
     <group name="${prefix}${name}_manipulator">
       <chain base_link="${prefix}base_link" tip_link="${prefix}tool0" />
+    </group>
+    <group name="${prefix}robotiq_gripper">
+      <joint name="${prefix}d435_mount_joint"/>
+      <joint name="${prefix}d435_mount_to_d435_joint"/>
+      <joint name="${prefix}d435_to_camera_wrist_joint"/>
+      <joint name="${prefix}d435_to_d435_inter_joint"/>
+      <joint name="${prefix}d435_to_wrist_optical_joint"/>
+      <joint name="${prefix}robotiq_coupler_joint"/>
+      <joint name="${prefix}robotiq_85_base_joint"/>
+      <joint name="${prefix}robotiq_85_left_inner_knuckle_joint"/>
+      <joint name="${prefix}robotiq_85_left_knuckle_joint"/>
+      <joint name="${prefix}robotiq_85_left_finger_joint"/>
+      <joint name="${prefix}robotiq_85_left_finger_tip_joint"/>
+      <joint name="${prefix}robotiq_85_right_inner_knuckle_joint"/>
+      <joint name="${prefix}robotiq_85_right_knuckle_joint"/>
+      <joint name="${prefix}robotiq_85_right_finger_joint"/>
+      <joint name="${prefix}robotiq_85_right_finger_tip_joint"/>
     </group>
     <!--GROUP STATES - Purpose - Define a named state for a particular group, in terms of joint values. This is useful to define states like 'folded arms'-->
@@ -39,5 +56,15 @@
       <joint name="${prefix}wrist_3_joint" value="-0.11" />
     </group_state>
+    <group_state name="${prefix}open" group="${prefix}robotiq_gripper">
+        <joint name="${prefix}robotiq_85_left_knuckle_joint" value="0"/>
+    </group_state>
+    <group_state name="${prefix}close_partial" group="${prefix}robotiq_gripper">
+        <joint name="${prefix}robotiq_85_left_knuckle_joint" value="0.6"/>
+    </group_state>
+    <group_state name="${prefix}close" group="${prefix}robotiq_gripper">
+        <joint name="${prefix}robotiq_85_left_knuckle_joint" value="0.8"/>
+    </group_state>
     <!--END EFFECTOR - Purpose - Represent information about an end effector.-->
+    <end_effector name="${prefix}robotiq_gripper" parent_link="${prefix}tool0" group="${prefix}robotiq_gripper"/>
     <!--VIRTUAL JOINT - Purpose - this element defines a virtual joint between a robot link and an external frame of reference (considered fixed with respect to the robot)-->
     <!--DISABLE COLLISIONS - By default it is assumed that any link of the robot could potentially come into collision with any other link in the robot. This tag disables collision checking between a specified pair of links. -->
@@ -53,4 +80,106 @@
     <disable_collisions link1="${prefix}wrist_1_link" link2="${prefix}wrist_3_link" reason="Never" />
     <disable_collisions link1="${prefix}wrist_2_link" link2="${prefix}wrist_3_link" reason="Adjacent" />
+    <disable_collisions link1="${prefix}d435" link2="${prefix}d435_mount_link" reason="Adjacent"/>
+    <disable_collisions link1="${prefix}d435" link2="${prefix}robotiq_85_base_link" reason="Never"/>
+    <disable_collisions link1="${prefix}d435" link2="${prefix}robotiq_85_left_finger_link" reason="Never"/>
+    <disable_collisions link1="${prefix}d435" link2="${prefix}robotiq_85_left_finger_tip_link" reason="Never"/>
+    <disable_collisions link1="${prefix}d435" link2="${prefix}robotiq_85_left_inner_knuckle_link" reason="Never"/>
+    <disable_collisions link1="${prefix}d435" link2="${prefix}robotiq_85_left_knuckle_link" reason="Never"/>
+    <disable_collisions link1="${prefix}d435" link2="${prefix}robotiq_85_right_finger_link" reason="Never"/>
+    <disable_collisions link1="${prefix}d435" link2="${prefix}robotiq_85_right_finger_tip_link" reason="Never"/>
+    <disable_collisions link1="${prefix}d435" link2="${prefix}robotiq_85_right_inner_knuckle_link" reason="Never"/>
+    <disable_collisions link1="${prefix}d435" link2="${prefix}robotiq_85_right_knuckle_link" reason="Never"/>
+    <disable_collisions link1="${prefix}d435" link2="${prefix}robotiq_coupler" reason="Never"/>
+    <disable_collisions link1="${prefix}d435" link2="wrist_1_link" reason="Never"/>
+    <disable_collisions link1="${prefix}d435" link2="wrist_2_link" reason="Never"/>
+    <disable_collisions link1="${prefix}d435" link2="wrist_3_link" reason="Never"/>
+    <disable_collisions link1="${prefix}d435_mount_link" link2="${prefix}robotiq_85_base_link" reason="Never"/>
+    <disable_collisions link1="${prefix}d435_mount_link" link2="${prefix}robotiq_85_left_finger_link" reason="Never"/>
+    <disable_collisions link1="${prefix}d435_mount_link" link2="${prefix}robotiq_85_left_finger_tip_link" reason="Never"/>
+    <disable_collisions link1="${prefix}d435_mount_link" link2="${prefix}robotiq_85_left_inner_knuckle_link" reason="Never"/>
+    <disable_collisions link1="${prefix}d435_mount_link" link2="${prefix}robotiq_85_left_knuckle_link" reason="Never"/>
+    <disable_collisions link1="${prefix}d435_mount_link" link2="${prefix}robotiq_85_right_finger_link" reason="Never"/>
+    <disable_collisions link1="${prefix}d435_mount_link" link2="${prefix}robotiq_85_right_finger_tip_link" reason="Never"/>
+    <disable_collisions link1="${prefix}d435_mount_link" link2="${prefix}robotiq_85_right_inner_knuckle_link" reason="Never"/>
+    <disable_collisions link1="${prefix}d435_mount_link" link2="${prefix}robotiq_85_right_knuckle_link" reason="Never"/>
+    <disable_collisions link1="${prefix}d435_mount_link" link2="${prefix}robotiq_coupler" reason="Adjacent"/>
+    <disable_collisions link1="${prefix}d435_mount_link" link2="wrist_1_link" reason="Never"/>
+    <disable_collisions link1="${prefix}d435_mount_link" link2="wrist_2_link" reason="Never"/>
+    <disable_collisions link1="${prefix}d435_mount_link" link2="wrist_3_link" reason="Adjacent"/>
+    <disable_collisions link1="${prefix}robotiq_85_base_link" link2="${prefix}robotiq_85_left_finger_link" reason="Never"/>
+    <disable_collisions link1="${prefix}robotiq_85_base_link" link2="${prefix}robotiq_85_left_finger_tip_link" reason="Never"/>
+    <disable_collisions link1="${prefix}robotiq_85_base_link" link2="${prefix}robotiq_85_left_inner_knuckle_link" reason="Adjacent"/>
+    <disable_collisions link1="${prefix}robotiq_85_base_link" link2="${prefix}robotiq_85_left_knuckle_link" reason="Adjacent"/>
+    <disable_collisions link1="${prefix}robotiq_85_base_link" link2="${prefix}robotiq_85_right_finger_link" reason="Never"/>
+    <disable_collisions link1="${prefix}robotiq_85_base_link" link2="${prefix}robotiq_85_right_finger_tip_link" reason="Never"/>
+    <disable_collisions link1="${prefix}robotiq_85_base_link" link2="${prefix}robotiq_85_right_inner_knuckle_link" reason="Adjacent"/>
+    <disable_collisions link1="${prefix}robotiq_85_base_link" link2="${prefix}robotiq_85_right_knuckle_link" reason="Adjacent"/>
+    <disable_collisions link1="${prefix}robotiq_85_base_link" link2="${prefix}robotiq_coupler" reason="Adjacent"/>
+    <disable_collisions link1="${prefix}robotiq_85_base_link" link2="wrist_1_link" reason="Never"/>
+    <disable_collisions link1="${prefix}robotiq_85_base_link" link2="wrist_2_link" reason="Never"/>
+    <disable_collisions link1="${prefix}robotiq_85_base_link" link2="wrist_3_link" reason="Never"/>
+    <disable_collisions link1="${prefix}robotiq_85_left_finger_link" link2="${prefix}robotiq_85_left_finger_tip_link" reason="Adjacent"/>
+    <disable_collisions link1="${prefix}robotiq_85_left_finger_link" link2="${prefix}robotiq_85_left_inner_knuckle_link" reason="Never"/>
+    <disable_collisions link1="${prefix}robotiq_85_left_finger_link" link2="${prefix}robotiq_85_left_knuckle_link" reason="Adjacent"/>
+    <disable_collisions link1="${prefix}robotiq_85_left_finger_link" link2="${prefix}robotiq_85_right_finger_link" reason="Never"/>
+    <disable_collisions link1="${prefix}robotiq_85_left_finger_link" link2="${prefix}robotiq_85_right_finger_tip_link" reason="Never"/>
+    <disable_collisions link1="${prefix}robotiq_85_left_finger_link" link2="${prefix}robotiq_85_right_inner_knuckle_link" reason="Never"/>
+    <disable_collisions link1="${prefix}robotiq_85_left_finger_link" link2="${prefix}robotiq_85_right_knuckle_link" reason="Never"/>
+    <disable_collisions link1="${prefix}robotiq_85_left_finger_link" link2="${prefix}robotiq_coupler" reason="Never"/>
+    <disable_collisions link1="${prefix}robotiq_85_left_finger_link" link2="wrist_1_link" reason="Never"/>
+    <disable_collisions link1="${prefix}robotiq_85_left_finger_link" link2="wrist_2_link" reason="Never"/>
+    <disable_collisions link1="${prefix}robotiq_85_left_finger_link" link2="wrist_3_link" reason="Never"/>
+    <disable_collisions link1="${prefix}robotiq_85_left_finger_tip_link" link2="${prefix}robotiq_85_left_inner_knuckle_link" reason="Default"/>
+    <disable_collisions link1="${prefix}robotiq_85_left_finger_tip_link" link2="${prefix}robotiq_85_left_knuckle_link" reason="Never"/>
+    <disable_collisions link1="${prefix}robotiq_85_left_finger_tip_link" link2="${prefix}robotiq_85_right_finger_link" reason="Never"/>
+    <disable_collisions link1="${prefix}robotiq_85_left_finger_tip_link" link2="${prefix}robotiq_85_right_finger_tip_link" reason="Never"/>
+    <disable_collisions link1="${prefix}robotiq_85_left_finger_tip_link" link2="${prefix}robotiq_85_right_inner_knuckle_link" reason="Never"/>
+    <disable_collisions link1="${prefix}robotiq_85_left_finger_tip_link" link2="${prefix}robotiq_85_right_knuckle_link" reason="Never"/>
+    <disable_collisions link1="${prefix}robotiq_85_left_finger_tip_link" link2="${prefix}robotiq_coupler" reason="Never"/>
+    <disable_collisions link1="${prefix}robotiq_85_left_finger_tip_link" link2="wrist_1_link" reason="Never"/>
+    <disable_collisions link1="${prefix}robotiq_85_left_finger_tip_link" link2="wrist_2_link" reason="Never"/>
+    <disable_collisions link1="${prefix}robotiq_85_left_finger_tip_link" link2="wrist_3_link" reason="Never"/>
+    <disable_collisions link1="${prefix}robotiq_85_left_inner_knuckle_link" link2="${prefix}robotiq_85_left_knuckle_link" reason="Never"/>
+    <disable_collisions link1="${prefix}robotiq_85_left_inner_knuckle_link" link2="${prefix}robotiq_85_right_finger_link" reason="Never"/>
+    <disable_collisions link1="${prefix}robotiq_85_left_inner_knuckle_link" link2="${prefix}robotiq_85_right_finger_tip_link" reason="Never"/>
+    <disable_collisions link1="${prefix}robotiq_85_left_inner_knuckle_link" link2="${prefix}robotiq_85_right_inner_knuckle_link" reason="Never"/>
+    <disable_collisions link1="${prefix}robotiq_85_left_inner_knuckle_link" link2="${prefix}robotiq_85_right_knuckle_link" reason="Never"/>
+    <disable_collisions link1="${prefix}robotiq_85_left_inner_knuckle_link" link2="${prefix}robotiq_coupler" reason="Never"/>
+    <disable_collisions link1="${prefix}robotiq_85_left_inner_knuckle_link" link2="wrist_1_link" reason="Never"/>
+    <disable_collisions link1="${prefix}robotiq_85_left_inner_knuckle_link" link2="wrist_2_link" reason="Never"/>
+    <disable_collisions link1="${prefix}robotiq_85_left_inner_knuckle_link" link2="wrist_3_link" reason="Never"/>
+    <disable_collisions link1="${prefix}robotiq_85_left_knuckle_link" link2="${prefix}robotiq_85_right_finger_link" reason="Never"/>
+    <disable_collisions link1="${prefix}robotiq_85_left_knuckle_link" link2="${prefix}robotiq_85_right_finger_tip_link" reason="Never"/>
+    <disable_collisions link1="${prefix}robotiq_85_left_knuckle_link" link2="${prefix}robotiq_85_right_inner_knuckle_link" reason="Never"/>
+    <disable_collisions link1="${prefix}robotiq_85_left_knuckle_link" link2="${prefix}robotiq_85_right_knuckle_link" reason="Never"/>
+    <disable_collisions link1="${prefix}robotiq_85_left_knuckle_link" link2="${prefix}robotiq_coupler" reason="Never"/>
+    <disable_collisions link1="${prefix}robotiq_85_left_knuckle_link" link2="wrist_1_link" reason="Never"/>
+    <disable_collisions link1="${prefix}robotiq_85_left_knuckle_link" link2="wrist_2_link" reason="Never"/>
+    <disable_collisions link1="${prefix}robotiq_85_left_knuckle_link" link2="wrist_3_link" reason="Never"/>
+    <disable_collisions link1="${prefix}robotiq_85_right_finger_link" link2="${prefix}robotiq_85_right_finger_tip_link" reason="Adjacent"/>
+    <disable_collisions link1="${prefix}robotiq_85_right_finger_link" link2="${prefix}robotiq_85_right_inner_knuckle_link" reason="Never"/>
+    <disable_collisions link1="${prefix}robotiq_85_right_finger_link" link2="${prefix}robotiq_85_right_knuckle_link" reason="Adjacent"/>
+    <disable_collisions link1="${prefix}robotiq_85_right_finger_link" link2="${prefix}robotiq_coupler" reason="Never"/>
+    <disable_collisions link1="${prefix}robotiq_85_right_finger_link" link2="wrist_1_link" reason="Never"/>
+    <disable_collisions link1="${prefix}robotiq_85_right_finger_link" link2="wrist_2_link" reason="Never"/>
+    <disable_collisions link1="${prefix}robotiq_85_right_finger_link" link2="wrist_3_link" reason="Never"/>
+    <disable_collisions link1="${prefix}robotiq_85_right_finger_tip_link" link2="${prefix}robotiq_85_right_inner_knuckle_link" reason="Default"/>
+    <disable_collisions link1="${prefix}robotiq_85_right_finger_tip_link" link2="${prefix}robotiq_85_right_knuckle_link" reason="Never"/>
+    <disable_collisions link1="${prefix}robotiq_85_right_finger_tip_link" link2="${prefix}robotiq_coupler" reason="Never"/>
+    <disable_collisions link1="${prefix}robotiq_85_right_finger_tip_link" link2="wrist_1_link" reason="Never"/>
+    <disable_collisions link1="${prefix}robotiq_85_right_finger_tip_link" link2="wrist_2_link" reason="Never"/>
+    <disable_collisions link1="${prefix}robotiq_85_right_finger_tip_link" link2="wrist_3_link" reason="Never"/>
+    <disable_collisions link1="${prefix}robotiq_85_right_inner_knuckle_link" link2="${prefix}robotiq_85_right_knuckle_link" reason="Never"/>
+    <disable_collisions link1="${prefix}robotiq_85_right_inner_knuckle_link" link2="${prefix}robotiq_coupler" reason="Never"/>
+    <disable_collisions link1="${prefix}robotiq_85_right_inner_knuckle_link" link2="wrist_1_link" reason="Never"/>
+    <disable_collisions link1="${prefix}robotiq_85_right_inner_knuckle_link" link2="wrist_2_link" reason="Never"/>
+    <disable_collisions link1="${prefix}robotiq_85_right_inner_knuckle_link" link2="wrist_3_link" reason="Never"/>
+    <disable_collisions link1="${prefix}robotiq_85_right_knuckle_link" link2="${prefix}robotiq_coupler" reason="Never"/>
+    <disable_collisions link1="${prefix}robotiq_85_right_knuckle_link" link2="wrist_1_link" reason="Never"/>
+    <disable_collisions link1="${prefix}robotiq_85_right_knuckle_link" link2="wrist_2_link" reason="Never"/>
+    <disable_collisions link1="${prefix}robotiq_85_right_knuckle_link" link2="wrist_3_link" reason="Never"/>
+    <disable_collisions link1="${prefix}robotiq_coupler" link2="wrist_1_link" reason="Never"/>
+    <disable_collisions link1="${prefix}robotiq_coupler" link2="wrist_2_link" reason="Never"/>
+    <disable_collisions link1="${prefix}robotiq_coupler" link2="wrist_3_link" reason="Never"/>
   </xacro:macro>
 </robot>

Commit message: add study start state

File: ur_moveit_config/srdf/ur_macro.srdf.xacro (robot description, xacro)
@@ -55,4 +55,12 @@
       <joint name="${prefix}wrist_2_joint" value="-1.6" />
       <joint name="${prefix}wrist_3_joint" value="-0.11" />
+    </group_state>
+    <group_state name="${prefix}study_home" group="${prefix}${name}_manipulator">
+      <joint name="${prefix}elbow_joint" value="2.5024" />
+      <joint name="${prefix}shoulder_lift_joint" value="-2.5486" />
+      <joint name="${prefix}shoulder_pan_joint" value="3.0716" />
+      <joint name="${prefix}wrist_1_joint" value="-2.2235" />
+      <joint name="${prefix}wrist_2_joint" value="-1.5846" />
+      <joint name="${prefix}wrist_3_joint" value="1.5600" />
     </group_state>
     <group_state name="${prefix}open" group="${prefix}robotiq_gripper">

Commit message: add look states

File: ur_moveit_config/srdf/ur_macro.srdf.xacro (robot description, xacro)
@@ -63,4 +63,20 @@
       <joint name="${prefix}wrist_2_joint" value="-1.5846" />
       <joint name="${prefix}wrist_3_joint" value="1.5600" />
+    </group_state>
+    <group_state name="${prefix}look_left" group="${prefix}${name}_manipulator">
+      <joint name="${prefix}elbow_joint" value="2.5024" />
+      <joint name="${prefix}shoulder_lift_joint" value="-2.5486" />
+      <joint name="${prefix}shoulder_pan_joint" value="3.0716" />
+      <joint name="${prefix}wrist_1_joint" value="-1.700" />
+      <joint name="${prefix}wrist_2_joint" value="-1.0332" />
+      <joint name="${prefix}wrist_3_joint" value="0.6822" />
+    </group_state>
+    <group_state name="${prefix}look_right" group="${prefix}${name}_manipulator">
+      <joint name="${prefix}elbow_joint" value="2.5024" />
+      <joint name="${prefix}shoulder_lift_joint" value="-2.5486" />
+      <joint name="${prefix}shoulder_pan_joint" value="3.0716" />
+      <joint name="${prefix}wrist_1_joint" value="-1.8598" />
+      <joint name="${prefix}wrist_2_joint" value="-2.1564" />
+      <joint name="${prefix}wrist_3_joint" value="3.0712" />
     </group_state>
     <group_state name="${prefix}open" group="${prefix}robotiq_gripper">
